File: indicador_led/indicador_led.kicad_sch (KiCad schematic)
At the start: 3 parts, among them J1 Conn_01x02_Pin

Commit message: ocultando token
Parts:
- R1: value R -> 1k
Changed lines of the file:
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@@
 			)
 		)
-		(property "Value" "R"
+		(property "Value" "1k"
 			(at 107.95 102.8699 0)
 			(show_name no)
